File: KiCad/TK3000/TK3000.kicad_pcb (KiCad board)
At the start: 2 copper layers, 239.6 x 239.9 mm, 316 parts, among them J12 Conn_01x01_Pin, J13 J13, J14 Power Connector, J16 J16, J17 J17, J18 Alto-Falante, J19 Conn_01x02_Pin, J8 DE9_Socket, J9 EAR/MIC, Q2 BC558, Q3 BC548, Q4 BF494, Q5 BC548, Q6 BC548, Q7 BC558, Y1 Crystal_Small

Commit message: Ajustes no silk e valores dos componentes
Parts:
- added C98: ??uF, TK3000:CP_Disc_5.08, F.Cu at (35.6, 246.8)
- JP11: value SolderJumper_2_Open -> X11
- moved C100 0.25 mm to (39.4, 259.3)
Routing:
- net +5V: track 1192.5 -> 1117.3 mm
Other:
- board text added: "16"
- board text added: "30"
- board text added: "31"
- board text added: "60"
- board text added: "M"
- board text added: "O"
- board text added: "R"
