File: KiCad/TK3000/TK3000.kicad_pcb (KiCad board)
At the start: 2 copper layers, 239.6 x 239.9 mm, 317 parts, among them J12 Conn_01x01_Pin, J13 J13, J14 Power Connector, J16 J16, J17 J17, J18 Alto-Falante, J19 Conn_01x02_Pin, J8 DE9_Socket, J9 EAR/MIC, Q2 BC558, Q3 BC548, Q4 BF494, Q5 BC548, Q6 BC548, Q7 BC558, X1 SolderJumper_2_Open, X11 X11, X12 SolderJumper_2_Bridged, X15 SolderJumper_2_Open, X16 SolderJumper_2_Bridged, X19 X19_X20, X2 SolderJumper_2_Bridged, X21 X21_X22, X23 SolderJumper_2_Open, X24 SolderJumper_2_Open, X25 Jumper_2_Open, X27 SolderJumper_2_Open, X3 SolderJumper_2_Open, X4 SolderJumper_2_Bridged, X5 SolderJumper_2_Open, X7 Jumper_2_Open, X9 SolderJumper_2_Open, Y1 Crystal_Small

Commit message: Ajustes em footprint
Parts:
- UE13: footprint Package_DIP:DIP-28_W15.24mm -> TK3000:DIP-28_W15.24mm
- UE15: footprint Package_DIP:DIP-40_W15.24mm -> TK3000:DIP-40_W15.24mm
