File: KiCad/TK3000/TK3000.kicad_pcb (KiCad board)
At the start: 2 copper layers, 239.6 x 239.9 mm, 319 parts, among them J10 EAR, J12 Conn_01x01_Pin, J13 J13, J14 Power Connector, J16 J16, J17 J17, J18 Alto-Falante, J19 Conn_01x02_Pin, J8 DE9_Socket, J9 EAR/MIC, Q2 BC558, Q3 BC548, Q4 BF494, Q5 BC548, Q6 BC548, Q7 BC558, X1 SolderJumper_2_Open, X11 X11, X12 SolderJumper_2_Bridged, X15 SolderJumper_2_Open, X16 SolderJumper_2_Bridged, X19 X19_X20, X2 SolderJumper_2_Bridged, X21 X21_X22, X23 SolderJumper_2_Open, X24 SolderJumper_2_Open, X25 Jumper_2_Open, X27 SolderJumper_2_Open, X3 SolderJumper_2_Open, X4 SolderJumper_2_Bridged, X5 SolderJumper_2_Open, X7 Jumper_2_Open, X9 SolderJumper_2_Open, Y1 Crystal_Small

Commit message: Atualização de valores dos componentes
Parts:
- C10, C11, C12, C13: value Capacitor -> 22nF
- C111: value Capacitor_Eletrolitico -> 10uF
- C120, C14, C87: value Capacitor -> C
- C2, C208, C4, C6, C8: value Capacitor -> 100nF
- C94, C95: value Capacitor -> 100pF
- C99: value Capacitor -> 33pF
- L4: value 27uH -> 47uH
- R100, R101, R109, R110, R115, R117, R97, R98, R99: value R -> 1k
- R102, R104, R105, R106, R45: value R -> 2k2
- R103, R73: value R -> 22k
- R11: value ~ -> 100R
- R119, R79, R95: value ~ -> 47R
- R3, R4, R5, R6, R7: value R -> 100R
- R33: value R -> 4k7
- R41: value 1k5 -> 1k
- R8: value R -> 12k
- R80: value ~ -> 22k
- UC13: value 74LS74_C13 -> 74LS74
- UE11: value 74LS74_E11 -> 74LS74
- UF10: value 74LS00_F10 -> 74LS00
- UF7: value 27C64_F7 -> 27C64
- UF9: value 74LS86_F9 -> 74LS86
- UH8: value 74LS166_H8 -> 74LS166
- X21: value X21_X22 -> X22
- Y1: value Crystal_Small -> 14.30244 MHz
