File: KiCad/TK3000/TK3000.kicad_sch (KiCad schematic)
At the start: 245 parts, among them J12 Conn_01x01_Pin, J13 J13, J14 Power Connector, J16 J16, J17 J17, J18 Alto-Falante, J19 Conn_01x02_Pin, J8 DE9_Socket, J9 EAR/MIC, Q2 BC558, Q3 BC548, Q4 BF494, Q5 BC548, Q6 BC548, Q7 BC558, Y1 Crystal_Small

Commit message: Ajustes no silk e valores dos componentes
Parts:
- C100, C101: value Capacitor -> 100nF
- JP11: value SolderJumper_2_Open -> X11
- R1: value R -> 220R
- R118, R30, R90, R91, R92, R93: value R -> 1k
- R17: value ~ -> 220R
- R18: value ~ -> 1k
- R19: value ~ -> 47R
- R2: value R -> 100R/1W
- R21: value 330 -> 220R
- R36: value R -> 2k2
- R76: value R -> 75R
- R77: value R -> 51k
- R78: value R -> 3k3
Other:
- company: (none) -> Clemar Folly Jr. - https://x.com/clemarfolly - https://facebook.com/clemarjr
- title: (none) -> Microdigital TK 3000 IIe
Changed lines of the file:
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@@
 	(generator_version "9.0")
 	(paper "A1")
+	(title_block
+		(title "Microdigital TK 3000 IIe")
+		(date "2026-09-02")
+		(rev "0 - Beta")
+		(company "Clemar Folly Jr. - https://x.com/clemarfolly - https://facebook.com/clemarjr")
+		(comment 1 "Recriado Por")
+		(comment 2 "em breve")
+		(comment 3 "Disponível em")
+	)
 	(rectangle
 		(start 284.226 151.892)
@@
 			)
 		)
-		(property "Value" "~"
-			(at 582.676 320.548 0)
+		(property "Value" "220R"
+			(at 584.708 320.548 90)
 			(effects
 				(font
@@
 			)
 		)
-		(property "Value" "R"
-			(at 184.15 451.6389 0)
+		(property "Value" "1k"
+			(at 180.594 455.93 90)
 			(effects
 				(font
@@
 				)
 				(justify left)
-				(hide yes)
 			)
 		)
@@
 			)
 		)
-		(property "Value" "R"
-			(at 180.34 451.6389 0)
+		(property "Value" "1k"
+			(at 176.53 455.93 90)
 			(effects
 				(font
@@
 				)
 				(justify left)
-				(hide yes)
 			)
 		)
@@
 			)
 		)
-		(property "Value" "Capacitor"
-			(at 523.2463 167.64 90)
+		(property "Value" "100nF"
+			(at 523.494 174.244 90)
 			(effects
 				(font
 					(size 1.27 1.27)
 				)
-				(hide yes)
 			)
 		)
@@
 		)
 		(property "Value" "1N914"
-			(at 533.908 170.434 0)
+			(at 530.606 179.07 90)
 			(effects
 				(font
 					(size 1.27 1.27)
 				)
-				(hide yes)
 			)
 		)
@@
 			)
 		)
-		(property "Value" "R"
-			(at 545.6189 167.64 0)
+		(property "Value" "75R"
+			(at 544.83 167.386 90)
 			(effects
 				(font
@@
 				)
 				(justify left)
-				(hide yes)
 			)
 		)
@@
 			)
 		)
-		(property "Value" "R"
-			(at 370.84 234.4689 0)
+		(property "Value" "2k2"
+			(at 378.206 236.728 0)
 			(effects
 				(font
@@
 				)
 				(justify left)
-				(hide yes)
 			)
 		)
@@
 			)
 		)
-		(property "Value" "Capacitor"
-			(at 547.37 167.6463 90)
+		(property "Value" "100nF"
+			(at 556.514 173.228 0)
 			(effects
 				(font
 					(size 1.27 1.27)
 				)
-				(hide yes)
 			)
 		)
@@
 			)
 		)
-		(property "Value" "R"
-			(at 384.81 384.3289 0)
+		(property "Value" "1k"
+			(at 383.794 385.572 0)
 			(effects
 				(font
@@
 				)
 				(justify left)
-				(hide yes)
 			)
 		)
@@
 			)
 		)
-		(property "Value" "R"
-			(at 191.77 451.6389 0)
+		(property "Value" "1k"
+			(at 188.214 455.93 90)
 			(effects
 				(font
@@
 				)
 				(justify left)
-				(hide yes)
 			)
 		)
@@
 			)
 		)
-		(property "Value" "~"
+		(property "Value" "1k"
 			(at 574.802 295.656 0)
 			(effects
@@
 			)
 		)
-		(property "Value" "R"
-			(at 218.44 118.8989 0)
+		(property "Value" "1k"
+			(at 224.536 119.888 0)
 			(effects
 				(font
@@
 				)
 				(justify left)
-				(hide yes)
 			)
 		)
@@
 		(dnp no)
 		(property "Reference" "R2"
-			(at 592.074 220.98 0)
+			(at 590.804 217.678 0)
 			(effects
 				(font
@@
 			)
 		)
-		(property "Value" "R"
-			(at 584.2 220.4989 0)
+		(property "Value" "100R/1W"
+			(at 597.154 220.472 0)
 			(effects
 				(font
@@
 				)
 				(justify left)
-				(hide yes)
 			)
 		)
@@
 			)
 		)
-		(property "Value" "R"
-			(at 515.62 166.8511 0)
+		(property "Value" "3k3"
+			(at 523.24 165.608 0)
 			(effects
 				(font
@@
 				)
 				(justify left)
-				(hide yes)
 			)
 		)
@@
 			)
 		)
-		(property "Value" "R"
-			(at 598.17 216.6889 0)
+		(property "Value" "220R"
+			(at 607.568 218.948 0)
 			(effects
 				(font
@@
 				)
 				(justify left)
-				(hide yes)
 			)
 		)
@@
 		)
 		(property "Value" "1k"
-			(at 481.33 441.1711 0)
+			(at 488.696 440.69 0)
 			(effects
 				(font
@@
 				)
 				(justify left)
-				(hide yes)
 			)
 		)
@@
 			)
 		)
-		(property "Value" "R"
-			(at 187.96 451.6389 0)
+		(property "Value" "1k"
+			(at 184.404 455.93 90)
 			(effects
 				(font
@@
 				)
 				(justify left)
-				(hide yes)
 			)
 		)
@@
 			)
 		)
-		(property "Value" "~"
-			(at 581.406 301.498 0)
+		(property "Value" "47R"
+			(at 582.676 306.07 90)
 			(effects
 				(font
@@
 			)
 		)
-		(property "Value" "R"
-			(at 531.3411 173.99 0)
+		(property "Value" "51k"
+			(at 532.13 173.228 90)
 			(effects
 				(font
@@
 				)
 				(justify left)
-				(hide yes)
 			)
 		)
@@
 			)
 		)
-		(property "Value" "330"
+		(property "Value" "220R"
 			(at 610.362 348.996 0)
 			(effects
@@
 			)
 		)
-		(property "Value" "SolderJumper_2_Open"
+		(property "Value" "X11"
 			(at 201.93 124.4599 90)
 			(effects
@@
 		(dnp no)
 		(property "Reference" "Q5"
-			(at 544.576 168.148 0)
+			(at 544.068 174.752 0)
 			(effects
 				(font
@@
 		)
 		(property "Value" "BC548"
-			(at 534.924 167.386 0)
+			(at 544.068 176.53 0)
 			(effects
 				(font
