File: KiCad/TK3000/TK3000.kicad_sch (KiCad schematic)
At the start: 317 parts, among them J12 Conn_01x01_Pin, J13 J13, J14 Power Connector, J16 J16, J17 J17, J18 Alto-Falante, J19 Conn_01x02_Pin, J8 DE9_Socket, J9 EAR/MIC, Q2 BC558, Q3 BC548, Q4 BF494, Q5 BC548, Q6 BC548, Q7 BC558, X1 SolderJumper_2_Open, X11 X11, X12 SolderJumper_2_Bridged, X15 SolderJumper_2_Open, X16 SolderJumper_2_Bridged, X19 X19_X20, X2 SolderJumper_2_Bridged, X21 X21_X22, X23 SolderJumper_2_Open, X24 SolderJumper_2_Open, X25 Jumper_2_Open, X27 SolderJumper_2_Open, X3 SolderJumper_2_Open, X4 SolderJumper_2_Bridged, X5 SolderJumper_2_Open, X7 Jumper_2_Open, X9 SolderJumper_2_Open, Y1 Crystal_Small

Commit message: Inclusão de valores de alguns componentes
Parts:
- C36, C80, C81, C97: value Capacitor -> 220pF
- C45: value Capacitor -> 47pF
- L4: value Ind -> 27uH
- R108: value R -> 120R
- R120: value R -> 1k
- R34, R35, R44: value ~ -> 120R
- R71: value R -> 47R
- R72: value R -> 470R
- R80: value 22k -> ~
Changed lines of the file:
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@@
 	)
 	(junction
-		(at 281.94 302.26)
-		(diameter 0)
-		(color 0 0 0 0)
-	)
-	(junction
 		(at 93.98 494.03)
 		(diameter 0)
@@
 		)
 	)
-	(bus
-		(pts
-			(xy 281.94 265.43) (xy 281.94 302.26)
-		)
-		(stroke
-			(width 0)
-			(type default)
-		)
-	)
 	(wire
 		(pts
@@
 		)
 	)
-	(bus
-		(pts
-			(xy 281.94 302.26) (xy 323.85 302.26)
-		)
-		(stroke
-			(width 0)
-			(type default)
-		)
-	)
 	(wire
 		(pts
@@
 	(bus
 		(pts
-			(xy 257.81 302.26) (xy 281.94 302.26)
+			(xy 257.81 302.26) (xy 323.85 302.26)
 		)
 		(stroke
@@
 			)
 		)
-		(property "Value" "R"
-			(at 257.81 201.4489 0)
+		(property "Value" "120R"
+			(at 266.7 204.724 0)
 			(effects
 				(font
@@
 				)
 				(justify left)
-				(hide yes)
 			)
 		)
@@
 			)
 		)
-		(property "Value" "~"
-			(at 193.04 196.0611 0)
+		(property "Value" "120R"
+			(at 192.786 197.612 90)
 			(effects
 				(font
@@
 				)
 				(justify left)
-				(hide yes)
 			)
 		)
@@
 		(dnp no)
 		(property "Reference" "C97"
-			(at 189.23 201.168 90)
+			(at 188.976 201.422 90)
 			(effects
 				(font
@@
 			)
 		)
-		(property "Value" "Capacitor"
-			(at 193.04 203.2062 0)
+		(property "Value" "220pF"
+			(at 193.04 204.724 90)
 			(effects
 				(font
@@
 				)
 				(justify left)
-				(hide yes)
 			)
 		)
@@
 			)
 		)
-		(property "Value" "Capacitor"
-			(at 219.71 196.8562 0)
+		(property "Value" "220pF"
+			(at 219.71 201.676 90)
 			(effects
 				(font
@@
 				)
 				(justify left)
-				(hide yes)
 			)
 		)
@@
 			)
 		)
-		(property "Value" "~"
-			(at 214.63 187.4789 0)
+		(property "Value" "120R"
+			(at 217.932 181.102 90)
 			(effects
 				(font
@@
 				)
 				(justify left)
-				(hide yes)
 			)
 		)
@@
 			)
 		)
-		(property "Value" "R"
-			(at 535.4589 135.89 0)
+		(property "Value" "1k"
+			(at 535.4589 135.89 90)
 			(effects
 				(font
@@
 				)
 				(justify left)
-				(hide yes)
 			)
 		)
@@
 			)
 		)
-		(property "Value" "R"
-			(at 316.992 188.468 0)
+		(property "Value" "47R"
+			(at 324.866 187.198 0)
 			(effects
 				(font
@@
 				)
 				(justify left)
-				(hide yes)
 			)
 		)
@@
 		(dnp no)
 		(property "Reference" "R95"
-			(at 202.184 197.104 90)
+			(at 205.486 197.104 90)
 			(effects
 				(font
@@
 		(dnp no)
 		(property "Reference" "C95"
-			(at 308.61 150.368 0)
+			(at 306.832 151.13 90)
 			(effects
 				(font
@@
 			)
 		)
-		(property "Value" "~"
-			(at 219.71 187.4789 0)
+		(property "Value" "120R"
+			(at 220.218 186.182 90)
 			(effects
 				(font
@@
 				)
 				(justify left)
-				(hide yes)
 			)
 		)
@@
 			)
 		)
-		(property "Value" "22k"
+		(property "Value" "~"
 			(at 84.328 269.748 0)
 			(effects
@@
 			)
 		)
-		(property "Value" "R"
-			(at 304.292 165.862 0)
+		(property "Value" "470R"
+			(at 306.324 164.846 90)
 			(effects
 				(font
@@
 				)
 				(justify left)
-				(hide yes)
 			)
 		)
@@
 			)
 		)
-		(property "Value" "Capacitor"
-			(at 224.79 196.8562 0)
+		(property "Value" "220pF"
+			(at 224.79 200.406 90)
 			(effects
 				(font
@@
 				)
 				(justify left)
-				(hide yes)
 			)
 		)
@@
 		(dnp no)
 		(property "Reference" "L4"
-			(at 600.71 375.158 90)
+			(at 600.71 371.348 0)
 			(effects
 				(font
@@
 			)
 		)
-		(property "Value" "Ind"
-			(at 600.71 374.65 90)
+		(property "Value" "27uH"
+			(at 601.98 373.888 0)
 			(effects
 				(font
 					(size 1.27 1.27)
 				)
-				(hide yes)
 			)
 		)
@@
 		(dnp no)
 		(property "Reference" "C36"
-			(at 253.492 199.136 0)
+			(at 252.984 197.866 0)
 			(effects
 				(font
@@
 			)
 		)
-		(property "Value" "Capacitor"
-			(at 257.81 204.4762 0)
+		(property "Value" "220pF"
+			(at 251.968 199.644 0)
 			(effects
 				(font
@@
 				)
 				(justify left)
-				(hide yes)
 			)
 		)
@@
 			)
 		)
-		(property "Value" "Capacitor"
-			(at 576.072 375.92 0)
+		(property "Value" "47pF"
+			(at 581.152 374.65 0)
 			(effects
 				(font
@@
 				)
 				(justify left)
-				(hide yes)
 			)
 		)
