File: KiCad/TK3000/TK3000.kicad_sch (KiCad schematic)
At the start: 317 parts, among them J12 Conn_01x01_Pin, J13 J13, J14 Power Connector, J16 J16, J17 J17, J18 Alto-Falante, J19 Conn_01x02_Pin, J8 DE9_Socket, J9 EAR/MIC, Q2 BC558, Q3 BC548, Q4 BF494, Q5 BC548, Q6 BC548, Q7 BC558, X1 SolderJumper_2_Open, X11 X11, X12 SolderJumper_2_Bridged, X15 SolderJumper_2_Open, X16 SolderJumper_2_Bridged, X19 X19_X20, X2 SolderJumper_2_Bridged, X21 X21_X22, X23 SolderJumper_2_Open, X24 SolderJumper_2_Open, X25 Jumper_2_Open, X27 SolderJumper_2_Open, X3 SolderJumper_2_Open, X4 SolderJumper_2_Bridged, X5 SolderJumper_2_Open, X7 Jumper_2_Open, X9 SolderJumper_2_Open, Y1 Crystal_Small

Commit message: Organização da pasta e inclusão do Ear separado.
Parts:
- added J10: EAR, TK3000:EarJack, symbol TK3000:J2_Jack
- added X6: ~, TK3000:PinHeader_1x03_P2.54mm_Vertical, symbol TK3000:Jumper_3_Open
- C1, C110, C3, C46, C5, C7, C9, C98: value ??uF -> 10uF
- C112: value Capacitor -> 100nF
- J9: symbol TK3000:AudioJack2 -> TK3000:J2_Jack
- R20: value R -> 4k7
- R27: value R -> 220k
- R28: value R -> 10k
- R32: value R -> 1k
Connections:
- net GND: now also J9.2, J10.2, J10.3; no longer J9.1
- net at R7.2, R8.1: now also J9.1, J9.3, X6.1 (A); no longer C112.2, J9.2
- new net: C112.2, X6.2 (C)
- new net: J10.1, X6.3 (B)
