File: KiCad/TK3000/power.kicad_sch (KiCad schematic)
At the start: 2 parts

Commit message: Inclusão de novos componentes.
Parts:
- added C113: 100nF, TK3000:C_Disc_5.08, symbol TK3000:Capacitor
- added UC13: 74LS74_C13, TK3000:DIP-14_W7.62mm, symbol TK3000:74LS74_C13
Connections:
- net +5V: now also C113.1, UC13.14 (VCC)
- net GND: now also C113.2, UC13.7 (GND)

Commit message: Avanços no processo.
Parts:
- added C102, C103, C104, C105, C106, C107, C108, C109, C21, C23, C24, C25, C26, C27, C28, C37, C38, C39, C40, C41, C42, C43, C47, C48, C49, C50, C51, C52, C53, C55, C58, C59, C64, C65, C66, C67, C71, C72, C73, C74, C77, C78, C84, C86, C89, C90, C91, C92, C93: 100nF, TK3000:C_Disc_5.08_12.7mm, symbol TK3000:Capacitor
- added C110: ??uF, TK3000:C_Elet_C110, symbol TK3000:Capacitor_Eletrolitico
- added C22, C56, C76, C85: 100nF, TK3000:C_Disc_12.7mm, symbol TK3000:Capacitor
- added C29, C30, C31, C32, C33, C34, C35, C57: 100nF, TK3000:C_Disc_5.08, symbol TK3000:Capacitor
- added C46, C70, C83: ??uF, TK3000:C_Elet_Tipo2, symbol TK3000:Capacitor_Eletrolitico
- added C79, C82: ??uF, TK3000:C_Elet_111, symbol TK3000:Capacitor_Eletrolitico
- added UE10: 74LS32, TK3000:DIP-14_W7.62mm, symbol TK3000:74LS32_E9
- added UE11: 74LS74_E11, TK3000:DIP-14_W7.62mm, symbol TK3000:74LS74_E11
- added UE9: 74LS32_E9, TK3000:DIP-14_W7.62mm, symbol TK3000:74LS32_E9
- added UF10: 74LS00_F10, TK3000:DIP-14_W7.62mm, symbol TK3000:74LS00_F10
- added UF11: 74LS08_F11, TK3000:DIP-14_W7.62mm, symbol TK3000:74LS08_F11
- added UF2: 74S02_F2, TK3000:DIP-14_W7.62mm, symbol TK3000:74S02_F2
- added UF9: 74LS86_F9, TK3000:DIP-14_W7.62mm, symbol TK3000:74LS86_F9
- added UH1: 74S109_H1, TK3000:DIP-16_W7.62mm, symbol TK3000:74S109_H1
- UF1: value F1 -> ~
Connections:
- net GND: now also C102.2, C103.2, C104.2, C105.2, C106.2, C107.2, C108.2, C109.2, C110.2, C21.2, C22.2, C23.2, C24.2, C25.2, C26.2, C27.2, C28.2, C29.2, C30.2, C31.2, C32.2, C33.2, C34.2, C35.2, C37.2, C38.2, C39.2, C40.2, C41.2, C42.2, C43.2, C46.2, C47.1, C48.1, C49.2, C50.2, C51.2, C52.2, C53.1, C55.1, C56.2, C57.2, C58.2, C59.1, C64.1, C65.2, C66.1, C67.1, C70.2, C71.1, C72.2, C73.2, C74.1, C76.2, C77.1, C78.2, C79.2, C82.2, C83.2, C84.2, C85.2, C86.2, C89.1, C90.2, C91.2, C92.1, C93.2, UE10.7 (GND), UE11.7 (GND), UE9.7 (GND), UF10.7 (GND), UF11.7 (GND), UF2.7 (GND), UF9.7 (GND), UH1.8 (GND)
- net +5V renamed +5C
- net +5C: now also C102.1, C103.1, C104.1, C105.1, C106.1, C107.1, C108.1, C109.1, C110.1, C21.1, C22.1, C23.1, C24.1, C25.1, C26.1, C27.1, C28.1, C46.1, C55.2, C56.1, C57.1, C58.1, C59.2, C64.2, C65.1, C66.2, C67.2, C70.1, C71.2, C72.1, C73.1, C74.2, C76.1, C77.2, C78.1, C79.1, C82.1, C83.1, C84.1, C85.1, C86.1, C89.2, C90.1, C91.1, C92.2, C93.1, UE10.14 (VCC), UE11.14 (VCC), UE9.14 (VCC), UF10.14 (VCC), UF11.14 (VCC), UF2.14 (VCC), UF9.14 (VCC), UH1.16 (VCC)
- new net +12C: C47.2, C48.2, C49.1, C50.1, C51.1, C52.1, C53.2
- new net -12V: C29.1, C30.1, C31.1, C32.1, C33.1, C34.1, C35.1
- new net -5V: C37.1, C38.1, C39.1, C40.1, C41.1, C42.1, C43.1
Other:
- moved on the sheet: C113, C68, UC13C, UF1E

Commit message: Erros de DRC zerados.
Parts:
- added C69: 100nF, TK3000:C_Disc_5.08_12.7mm, symbol TK3000:Capacitor
- added C88: 100nF, TK3000:C_Disc_12.7mm, symbol TK3000:Capacitor
- C65: footprint TK3000:C_Disc_5.08_12.7mm -> TK3000:C65_Disc_5.08_12.7mm
- UE10: footprint TK3000:DIP-14_W7.62mm -> TK3000:UE10_DIP-14_W7.62mm
- UE11: footprint TK3000:DIP-14_W7.62mm -> TK3000:UE11_DIP-14_W7.62mm
- UE9: footprint TK3000:DIP-14_W7.62mm -> TK3000:UE9_DIP-14_W7.62mm
Connections:
- net +5C: no longer C102.1, C103.1, C104.1, C105.1, C106.1, C107.1, C108.1, C109.1, C110.1, C113.1, C21.1, C46.1, C55.2, C56.1, C57.1, C58.1, C59.2, C64.2, C65.1, C66.2, C67.2, C68.1, C70.1, C71.2, C72.1, C73.1, C74.2, C76.1, C77.2, C78.1, C79.1, C82.1, C83.1, C84.1, C85.1, C86.1, C89.2, C90.1, C91.1, C92.2, C93.1, UC13.14 (VCC), UE10.14 (VCC), UE11.14 (VCC), UE9.14 (VCC), UF1.14 (VCC), UF10.14 (VCC), UF11.14 (VCC), UF2.14 (VCC), UF9.14 (VCC), UH1.16 (VCC)
- net GND: now also C69.2, C88.1
- new net +5V: C102.1, C103.1, C104.1, C105.1, C106.1, C107.1, C108.1, C109.1, C110.1, C113.1, C21.1, C46.1, C55.2, C56.1, C57.1, C58.1, C59.2, C64.2, C65.1, C66.2, C67.2, C68.1, C69.1, C70.1, C71.2, C72.1, C73.1, C74.2, C76.1, C77.2, C78.1, C79.1, C82.1, C83.1, C84.1, C85.1, C86.1, C88.2, C89.2, C90.1, C91.1, C92.2, C93.1, UC13.14 (VCC), UE10.14 (VCC), UE11.14 (VCC), UE9.14 (VCC), UF1.14 (VCC), UF10.14 (VCC), UF11.14 (VCC), UF2.14 (VCC), UF9.14 (VCC), UH1.16 (VCC)
Other:
- moved on the sheet: C85, C86

Commit message: Ajustes no silk e valores dos componentes
Parts:
- added C98: ??uF, TK3000:CP_Disc_5.08, symbol TK3000:Capacitor_Eletrolitico
- C70, C79, C82, C83: value ??uF -> 10uF
Connections:
- net +5V: now also C98.1
- net GND: now also C98.2
Changed lines of the file:
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@@
 	(generator "eeschema")
 	(generator_version "9.0")
-	(paper "A4")
+	(paper "A1")
 	(junction
 		(at 27.94 173.99)
@@
 			)
 		)
-		(property "Value" "??uF"
+		(property "Value" "10uF"
 			(at 172.72 115.9509 0)
 			(effects
@@
 			)
 		)
-		(property "Value" "??uF"
+		(property "Value" "10uF"
 			(at 147.32 115.9509 0)
 			(effects
@@
 			)
 		)
-		(property "Value" "??uF"
+		(property "Value" "10uF"
 			(at 196.85 115.9509 0)
 			(effects
@@
 	)
 	(symbol
+		(lib_id "TK3000:Capacitor_Eletrolitico")
+		(at 217.17 115.57 0)
+		(unit 1)
+		(exclude_from_sim no)
+		(in_bom yes)
+		(on_board yes)
+		(dnp no)
+		(fields_autoplaced yes)
+		(property "Reference" "C98"
+			(at 220.98 113.4109 0)
+			(effects
+				(font
+					(size 1.27 1.27)
+				)
+				(justify left)
+			)
+		)
+		(property "Value" "??uF"
+			(at 220.98 115.9509 0)
+			(effects
+				(font
+					(size 1.27 1.27)
+				)
+				(justify left)
+			)
+		)
+		(property "Footprint" "TK3000:CP_Disc_5.08"
+			(at 218.1352 119.38 0)
+			(effects
+				(font
+					(size 1.27 1.27)
+				)
+				(hide yes)
+			)
+		)
+		(property "Datasheet" "~"
+			(at 217.17 115.57 0)
+			(effects
+				(font
+					(size 1.27 1.27)
+				)
+				(hide yes)
+			)
+		)
+		(property "Description" "Polarized capacitor"
+			(at 217.17 115.57 0)
+			(effects
+				(font
+					(size 1.27 1.27)
+				)
+				(hide yes)
+			)
+		)
+		(pin "2"
+		)
+		(pin "1"
+		)
+		(instances
+			(project "TK3000"
+				(path "/12cba11f-a914-4a6a-8e77-4856f6513f0b/8c52bed7-6241-4139-b05c-0297ba221d02"
+					(reference "C98")
+					(unit 1)
+				)
+			)
+		)
+	)
+	(symbol
 		(lib_id "power:+5V")
 		(at 120.65 71.12 0)
@@
 	(symbol
 		(lib_id "power:GND")
+		(at 217.17 119.38 0)
+		(unit 1)
+		(exclude_from_sim no)
+		(in_bom yes)
+		(on_board yes)
+		(dnp no)
+		(property "Reference" "#PWR0328"
+			(at 217.17 125.73 0)
+			(effects
+				(font
+					(size 1.27 1.27)
+				)
+				(hide yes)
+			)
+		)
+		(property "Value" "GND"
+			(at 217.17 123.19 0)
+			(effects
+				(font
+					(size 1.27 1.27)
+				)
+			)
+		)
+		(property "Footprint" ""
+			(at 217.17 119.38 0)
+			(effects
+				(font
+					(size 1.27 1.27)
+				)
+				(hide yes)
+			)
+		)
+		(property "Datasheet" ""
+			(at 217.17 119.38 0)
+			(effects
+				(font
+					(size 1.27 1.27)
+				)
+				(hide yes)
+			)
+		)
+		(property "Description" "Power symbol creates a global label with name \"GND\" , ground"
+			(at 217.17 119.38 0)
+			(effects
+				(font
+					(size 1.27 1.27)
+				)
+				(hide yes)
+			)
+		)
+		(pin "1"
+		)
+		(instances
+			(project "TK3000"
+				(path "/12cba11f-a914-4a6a-8e77-4856f6513f0b/8c52bed7-6241-4139-b05c-0297ba221d02"
+					(reference "#PWR0328")
+					(unit 1)
+				)
+			)
+		)
+	)
+	(symbol
+		(lib_id "power:GND")
 		(at 72.39 59.69 0)
 		(unit 1)
@@
 			)
 		)
-		(property "Value" "??uF"
+		(property "Value" "10uF"
 			(at 184.15 115.9509 0)
 			(effects
@@
 					(unit 1)
 				)
+			)
+		)
+	)
+	(symbol
+		(lib_id "power:+5V")
+		(at 217.17 111.76 0)
+		(unit 1)
+		(exclude_from_sim no)
+		(in_bom yes)
+		(on_board yes)
+		(dnp no)
+		(property "Reference" "#PWR0327"
+			(at 217.17 115.57 0)
+			(effects
+				(font
+					(size 1.27 1.27)
+				)
+				(hide yes)
+			)
+		)
+		(property "Value" "+5V"
+			(at 217.17 108.458 0)
+			(effects
+				(font
+					(size 1.27 1.27)
+				)
+			)
+		)
+		(property "Footprint" ""
+			(at 217.17 111.76 0)
+			(effects
+				(font
+					(size 1.27 1.27)
+				)
+				(hide yes)
+			)
+		)
+		(property "Datasheet" ""
+			(at 217.17 111.76 0)
+			(effects
+				(font
+					(size 1.27 1.27)
+				)
+				(hide yes)
+			)
+		)
+		(property "Description" "Power symbol creates a global label with name \"+5V\""
+			(at 217.17 111.76 0)
+			(effects
+				(font
+					(size 1.27 1.27)
+				)
+				(hide yes)
+			)
+		)
+		(pin "1"
+		)
+		(instances
+			(project "TK3000"
+				(path "/12cba11f-a914-4a6a-8e77-4856f6513f0b/8c52bed7-6241-4139-b05c-0297ba221d02"
+					(reference "#PWR0327")
+					(unit 1)
+				)
