File: KiCad/TK3000/_autosave-TK3000.kicad_sch (KiCad schematic)
At the start: 245 parts, among them J12 Conn_01x01_Pin, J13 J13, J14 Power Connector, J16 J16, J17 J17, J18 Alto-Falante, J19 Conn_01x02_Pin, J8 DE9_Socket, J9 EAR/MIC, Q2 BC558, Q3 BC548, Q4 BF494, Q5 BC548, Q6 BC548, Q7 BC558, Y1 Crystal_Small

Commit message: Ajustes na fonte ttf e no esquema.
Parts:
- added C102, C103, C104, C105, C106, C107, C108, C109, C21, C23, C24, C25, C26, C27, C28, C37, C38, C39, C40, C41, C42, C43, C47, C48, C49, C50, C51, C52, C53, C55, C58, C59, C64, C66, C67, C68, C69, C71, C72, C73, C74, C77, C78, C84, C86, C89, C90, C91, C92, C93: 100nF, TK3000:C_Disc_5.08_12.7mm, symbol TK3000:Capacitor
- added C110: ??uF, TK3000:C_Elet_C110, symbol TK3000:Capacitor_Eletrolitico
- added C113, C29, C30, C31, C32, C33, C34, C35, C57: 100nF, TK3000:C_Disc_5.08, symbol TK3000:Capacitor
- added C22, C56, C76, C85, C88: 100nF, TK3000:C_Disc_12.7mm, symbol TK3000:Capacitor
- added C46: ??uF, TK3000:C_Elet_Tipo2, symbol TK3000:Capacitor_Eletrolitico
- added C65: 100nF, TK3000:C65_Disc_5.08_12.7mm, symbol TK3000:Capacitor
- added C70, C83: 10uF, TK3000:C_Elet_Tipo2, symbol TK3000:Capacitor_Eletrolitico
- added C79, C82: 10uF, TK3000:C_Elet_111, symbol TK3000:Capacitor_Eletrolitico
- added C98: ??uF, TK3000:CP_Disc_5.08, symbol TK3000:Capacitor_Eletrolitico
- added unit 3 of UC13
- added unit 5 of UE10
- added unit 3 of UE11
- added unit 5 of UE9
- added unit 5 of UF1
- added unit 5 of UF10
- added unit 5 of UF11
- added unit 5 of UF2
- added unit 5 of UF9
- added unit 3 of UH1
- R41: value ~ -> 1k5
- R47, R48, R49, R54: value 3k3 -> 2k2
- UE13: footprint TK3000:DIP-28_W15.24mm -> Package_DIP:DIP-28_W15.24mm
- UE15: footprint TK3000:DIP-40_W15.24mm -> Package_DIP:DIP-40_W15.24mm
- UF1: value ~ -> 74LS125
- renumbered JP1 to X1, JP11 to X11, JP12 to X12, JP15 to X15, JP16 to X16, JP19 to X19, JP2 to X2, JP21 to X21, JP23 to X23, JP24 to X24, JP25 to X25, JP27 to X27, JP3 to X3, JP4 to X4, JP5 to X5, JP7 to X7, JP9 to X9
Connections:
- net +12C: now also C47.2, C48.2, C49.1, C50.1, C51.1, C52.1, C53.2
- net +5C: now also C22.1, C23.1, C24.1, C25.1, C26.1, C27.1, C28.1
- net +5V: now also C102.1, C103.1, C104.1, C105.1, C106.1, C107.1, C108.1, C109.1, C110.1, C113.1, C21.1, C46.1, C55.2, C56.1, C57.1, C58.1, C59.2, C64.2, C65.1, C66.2, C67.2, C68.1, C69.1, C70.1, C71.2, C72.1, C73.1, C74.2, C76.1, C77.2, C78.1, C79.1, C82.1, C83.1, C84.1, C85.1, C86.1, C88.2, C89.2, C90.1, C91.1, C92.2, C93.1, C98.1, UC13.14 (VCC), UE10.14 (VCC), UE11.14 (VCC), UE9.14 (VCC), UF1.14 (VCC), UF10.14 (VCC), UF11.14 (VCC), UF2.14 (VCC), UF9.14 (VCC), UH1.16 (VCC)
- net -12V: now also C29.1, C30.1, C31.1, C32.1, C33.1, C34.1, C35.1
- net -5V: now also C37.1, C38.1, C39.1, C40.1, C41.1, C42.1, C43.1
- net GND: now also C102.2, C103.2, C104.2, C105.2, C106.2, C107.2, C108.2, C109.2, C110.2, C113.2, C21.2, C22.2, C23.2, C24.2, C25.2, C26.2, C27.2, C28.2, C29.2, C30.2, C31.2, C32.2, C33.2, C34.2, C35.2, C37.2, C38.2, C39.2, C40.2, C41.2, C42.2, C43.2, C46.2, C47.1, C48.1, C49.2, C50.2, C51.2, C52.2, C53.1, C55.1, C56.2, C57.2, C58.2, C59.1, C64.1, C65.2, C66.1, C67.1, C68.2, C69.2, C70.2, C71.1, C72.2, C73.2, C74.1, C76.2, C77.1, C78.2, C79.2, C82.2, C83.2, C84.2, C85.2, C86.2, C88.1, C89.1, C90.2, C91.2, C92.1, C93.2, C98.2, UC13.7 (GND), UE10.7 (GND), UE11.7 (GND), UE9.7 (GND), UF1.7 (GND), UF10.7 (GND), UF11.7 (GND), UF2.7 (GND), UF9.7 (GND), UH1.8 (GND)
Other:
- removed sheet Power and Decoupling Caps
- moved on the sheet: J14, J8
